Commit message: fix frames

File: reacher/data/pupper_arm.urdf (robot description, URDF)
Before this commit: robot pupper_arm, 5 links, 4 joints
Joints:
- joint baseMotor: limit lower=-6 upper=6 effort=0 velocity=0 -> lower=-10 upper=10 effort=0 velocity=0; origin xyz=0 0 -0.025 rpy=1.5708 0 0 -> xyz=0 0 -0.025 rpy=1.5708 0 -1.5708
- joint leftFrontLowerLegMotor: limit lower=-6 upper=6 effort=0 velocity=0 -> lower=-10 upper=10 effort=0 velocity=0
- joint leftFrontUpperLegMotor: limit lower=-0.8 upper=6 effort=0 velocity=0 -> lower=-10 upper=10 effort=0 velocity=0
